File: KiCad/projecte_neteja_parabrises/Potencia.kicad_sch (KiCad schematic)
At the start: 0 parts

Commit message: Prueba Potencia
Parts:
- added J2: Conn_01x09_Pin, symbol Connector:Conn_01x09_Pin
Changed lines of the file:
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@@
 	(generator_version "9.0")
 	(paper "A4")
+	(symbol
+		(lib_id "Connector:Conn_01x09_Pin")
+		(at 137.16 78.105 0)
+		(unit 1)
+		(exclude_from_sim no)
+		(in_bom yes)
+		(on_board yes)
+		(dnp no)
+		(fields_autoplaced yes)
+		(property "Reference" "J2"
+			(at 137.795 63.5 0)
+			(effects
+				(font
+					(size 1.27 1.27)
+				)
+			)
+		)
+		(property "Value" "Conn_01x09_Pin"
+			(at 137.795 66.04 0)
+			(effects
+				(font
+					(size 1.27 1.27)
+				)
+			)
+		)
+		(property "Footprint" ""
+			(at 137.16 78.105 0)
+			(effects
+				(font
+					(size 1.27 1.27)
+				)
+				(hide yes)
+			)
+		)
+		(property "Datasheet" "~"
+			(at 137.16 78.105 0)
+			(effects
+				(font
+					(size 1.27 1.27)
+				)
+				(hide yes)
+			)
+		)
+		(property "Description" "Generic connector, single row, 01x09, script generated"
+			(at 137.16 78.105 0)
+			(effects
+				(font
+					(size 1.27 1.27)
+				)
+				(hide yes)
+			)
+		)
+		(pin "3"
+		)
+		(pin "4"
+		)
+		(pin "6"
+		)
+		(pin "5"
+		)
+		(pin "2"
+		)
+		(pin "1"
+		)
+		(pin "9"
+		)
+		(pin "8"
+		)
+		(pin "7"
+		)
+		(instances
+			(project ""
+				(path "/83fe8808-b70b-463e-9fcd-89556c9690a9/54835b05-573d-4299-97f2-a5366b1fd616"
+					(reference "J2")
+					(unit 1)
+				)
+			)
+		)
+	)
 )

Commit message: Potencia actualizada
Parts:
- removed J2: Conn_01x09_Pin, symbol Connector:Conn_01x09_Pin
- added D1: D, symbol Device:D
- added K2: EE2-3NKX, Relay_SMD:Relay_DPDT_Kemet_EE2_NUX_NKX, symbol Relay:EE2-3NKX
- added M1, M2, M3, M4: Motor_DC, symbol Motor:Motor_DC
- added Q1: NPN, symbol Simulation_SPICE:NPN
- added R1: R, symbol Device:R
- added U2, U3: DRV8871DDA, Package_SO:Texas_HTSOP-8-1EP_3.9x4.9mm_P1.27mm_EP2.95x4.9mm_Mask2.4x3.1mm_ThermalVias, symbol Driver_Motor:DRV8871DDA
Connections:
- new net: D1.1 (K), K2.1
- new net: D1.2 (A), K2.12, Q1.1 (C)
- new net: U2.1 (GND), U2.7 (GND), U2.9 (GND)
- new net: M1.1 (+), U2.6 (OUT1)
- new net: M1.2 (-), U2.8 (OUT2)
- new net: Q1.2 (B), R1.2
- new net: U3.1 (GND), U3.7 (GND), U3.9 (GND)
- new net: M2.1 (+), U3.6 (OUT1)
- new net: M2.2 (-), U3.8 (OUT2)
- new net: K2.8, M3.1 (+)
- new net: K2.5, M4.1 (+)
- new net GND: M3.2 (-), M4.2 (-), Q1.3 (E)
- new net VDD: K2.4, K2.9
- new net micro: R1.1

Commit message: micro
Parts:
- renumbered R1 to 1k, D1 to D?, K2 to K?, M1 to M?, M3 to M?, M4 to M?, M2 to M?, Q1 to Q?, U2 to U?, U3 to U?
Connections:
- net GND: now also U?.1 (GND), U?.1 (GND), U?.7 (GND), U?.7 (GND), U?.9 (GND), U?.9 (GND)
Changed lines of the file:
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@@
+	)
+	(symbol
+		(lib_id "power:GND")
+		(at 92.71 67.31 0)
+		(unit 1)
+		(exclude_from_sim no)
+		(in_bom yes)
+		(on_board yes)
+		(dnp no)
+		(fields_autoplaced yes)
+		(property "Reference" "#PWR02"
+			(at 92.71 73.66 0)
+			(effects
+				(font
+					(size 1.27 1.27)
+				)
+				(hide yes)
+			)
+		)
+		(property "Value" "GND"
+			(at 92.71 72.39 0)
+			(effects
+				(font
+					(size 1.27 1.27)
+				)
+			)
+		)
+		(property "Footprint" ""
+			(at 92.71 67.31 0)
+			(effects
+				(font
+					(size 1.27 1.27)
+				)
+				(hide yes)
+			)
+		)
+		(property "Datasheet" ""
+			(at 92.71 67.31 0)
+			(effects
+				(font
+					(size 1.27 1.27)
+				)
+				(hide yes)
+			)
+		)
+		(property "Description" "Power symbol creates a global label with name \"GND\" , ground"
+			(at 92.71 67.31 0)
+			(effects
+				(font
+					(size 1.27 1.27)
+				)
+				(hide yes)
+			)
+		)
+		(pin "1"
+		)
+		(instances
+			(project ""
+				(path "/82bf9682-9f8b-46a0-adc6-e19c50674fc0"
+					(reference "#PWR02")
+					(unit 1)
+				)
+			)
+		)
 	)
 	(symbol
@@
 		(dnp no)
 		(fields_autoplaced yes)
-		(property "Reference" "D1"
+		(property "Reference" "D?"
 			(at 114.3 101.5999 90)
 			(effects
@@
 		)
 		(instances
+			(project "Potencia"
+				(path "/82bf9682-9f8b-46a0-adc6-e19c50674fc0"
+					(reference "D?")
+					(unit 1)
+				)
+			)
 			(project ""
 				(path "/83fe8808-b70b-463e-9fcd-89556c9690a9/54835b05-573d-4299-97f2-a5366b1fd616"
@@
 		(dnp no)
 		(fields_autoplaced yes)
-		(property "Reference" "U2"
+		(property "Reference" "U?"
 			(at 94.8533 44.45 0)
 			(effects
@@
 		)
 		(instances
+			(project "Potencia"
+				(path "/82bf9682-9f8b-46a0-adc6-e19c50674fc0"
+					(reference "U?")
+					(unit 1)
+				)
+			)
 			(project ""
 				(path "/83fe8808-b70b-463e-9fcd-89556c9690a9/54835b05-573d-4299-97f2-a5366b1fd616"
@@
 		(dnp no)
 		(fields_autoplaced yes)
-		(property "Reference" "Q1"
+		(property "Reference" "Q?"
 			(at 128.905 116.2049 0)
 			(effects
@@
 		)
 		(instances
+			(project "Potencia"
+				(path "/82bf9682-9f8b-46a0-adc6-e19c50674fc0"
+					(reference "Q?")
+					(unit 1)
+				)
+			)
 			(project ""
 				(path "/83fe8808-b70b-463e-9fcd-89556c9690a9/54835b05-573d-4299-97f2-a5366b1fd616"
@@
 		(dnp no)
 		(fields_autoplaced yes)
-		(property "Reference" "M1"
+		(property "Reference" "M?"
 			(at 123.825 55.2449 0)
 			(effects
@@
 		)
 		(instances
+			(project "Potencia"
+				(path "/82bf9682-9f8b-46a0-adc6-e19c50674fc0"
+					(reference "M?")
+					(unit 1)
+				)
+			)
 			(project ""
 				(path "/83fe8808-b70b-463e-9fcd-89556c9690a9/54835b05-573d-4299-97f2-a5366b1fd616"
@@
 		(on_board yes)
 		(dnp no)
-		(property "Reference" "#PWR01"
+		(property "Reference" "#PWR?"
 			(at 157.48 84.455 0)
 			(effects
@@
 		)
 		(instances
+			(project "Potencia"
+				(path "/82bf9682-9f8b-46a0-adc6-e19c50674fc0"
+					(reference "#PWR?")
+					(unit 1)
+				)
+			)
 			(project ""
 				(path "/83fe8808-b70b-463e-9fcd-89556c9690a9/54835b05-573d-4299-97f2-a5366b1fd616"
@@
 		(dnp no)
 		(fields_autoplaced yes)
-		(property "Reference" "#PWR02"
+		(property "Reference" "#PWR?"
 			(at 167.64 92.075 0)
 			(effects
@@
 		)
 		(instances
+			(project "Potencia"
+				(path "/82bf9682-9f8b-46a0-adc6-e19c50674fc0"
+					(reference "#PWR?")
+					(unit 1)
+				)
+			)
 			(project ""
 				(path "/83fe8808-b70b-463e-9fcd-89556c9690a9/54835b05-573d-4299-97f2-a5366b1fd616"
@@
 		(dnp no)
 		(fields_autoplaced yes)
-		(property "Reference" "U3"
+		(property "Reference" "U?"
 			(at 146.9233 43.815 0)
 			(effects
@@
 		)
 		(instances
+			(project "Potencia"
+				(path "/82bf9682-9f8b-46a0-adc6-e19c50674fc0"
+					(reference "U?")
+					(unit 1)
+				)
+			)
 			(project "projecte_neteja_parabrises"
 				(path "/83fe8808-b70b-463e-9fcd-89556c9690a9/54835b05-573d-4299-97f2-a5366b1fd616"
@@
 		(on_board yes)
 		(dnp no)
-		(fields_autoplaced yes)
-		(property "Reference" "R1"
-			(at 114.3 111.76 90)
+		(property "Reference" "1k"
+			(at 114.935 122.555 90)
 			(effects
 				(font
@@
 		)
 		(instances
+			(project "Potencia"
+				(path "/82bf9682-9f8b-46a0-adc6-e19c50674fc0"
+					(reference "1k")
+					(unit 1)
+				)
+			)
 			(project ""
 				(path "/83fe8808-b70b-463e-9fcd-89556c9690a9/54835b05-573d-4299-97f2-a5366b1fd616"
@@
 		(on_board yes)
 		(dnp no)
-		(property "Reference" "M3"
+		(property "Reference" "M?"
 			(at 158.75 88.9 90)
 			(effects
@@
 		)
 		(instances
+			(project "Potencia"
+				(path "/82bf9682-9f8b-46a0-adc6-e19c50674fc0"
+					(reference "M?")
+					(unit 1)
+				)
+			)
 			(project ""
 				(path "/83fe8808-b70b-463e-9fcd-89556c9690a9/54835b05-573d-4299-97f2-a5366b1fd616"
@@
 		(dnp no)
 		(fields_autoplaced yes)
-		(property "Reference" "M4"
+		(property "Reference" "M?"
 			(at 146.05 76.2 90)
 			(effects
@@
 		)
 		(instances
+			(project "Potencia"
+				(path "/82bf9682-9f8b-46a0-adc6-e19c50674fc0"
+					(reference "M?")
+					(unit 1)
+				)
+			)
 			(project ""
 				(path "/83fe8808-b70b-463e-9fcd-89556c9690a9/54835b05-573d-4299-97f2-a5366b1fd616"
@@
 		(dnp no)
 		(fields_autoplaced yes)
-		(property "Reference" "K2"
+		(property "Reference" "K?"
 			(at 152.4 100.9649 0)
 			(effects
@@
 		)
 		(instances
+			(project "Potencia"
+				(path "/82bf9682-9f8b-46a0-adc6-e19c50674fc0"
+					(reference "K?")
+					(unit 1)
+				)
+			)
 			(project ""
 				(path "/83fe8808-b70b-463e-9fcd-89556c9690a9/54835b05-573d-4299-97f2-a5366b1fd616"
 					(reference "K2")
+					(unit 1)
+				)
+			)
+		)
+	)
+	(symbol
+		(lib_id "power:GND")
+		(at 144.78 66.675 0)
+		(unit 1)
+		(exclude_from_sim no)
+		(in_bom yes)
+		(on_board yes)
+		(dnp no)
+		(fields_autoplaced yes)
+		(property "Reference" "#PWR01"
+			(at 144.78 73.025 0)
+			(effects
+				(font
+					(size 1.27 1.27)
+				)
+				(hide yes)
+			)
+		)
+		(property "Value" "GND"
+			(at 144.78 71.12 0)
+			(effects
+				(font
+					(size 1.27 1.27)
+				)
+			)
+		)
+		(property "Footprint" ""
+			(at 144.78 66.675 0)
+			(effects
+				(font
+					(size 1.27 1.27)
+				)
+				(hide yes)
+			)
+		)
+		(property "Datasheet" ""
+			(at 144.78 66.675 0)
+			(effects
+				(font
+					(size 1.27 1.27)
+				)
+				(hide yes)
+			)
+		)
+		(property "Description" "Power symbol creates a global label with name \"GND\" , ground"
+			(at 144.78 66.675 0)
+			(effects
+				(font
+					(size 1.27 1.27)
+				)
+				(hide yes)
+			)
+		)
+		(pin "1"
+		)
+		(instances
+			(project ""
+				(path "/82bf9682-9f8b-46a0-adc6-e19c50674fc0"
+					(reference "#PWR01")
 					(unit 1)
 				)
@@
 		(dnp no)
 		(fields_autoplaced yes)
-		(property "Reference" "M2"
+		(property "Reference" "M?"
 			(at 178.435 53.9749 0)
 			(effects
@@
 		)
 		(instances
+			(project "Potencia"
+				(path "/82bf9682-9f8b-46a0-adc6-e19c50674fc0"
+					(reference "M?")
+					(unit 1)
+				)
+			)
 			(project ""
 				(path "/83fe8808-b70b-463e-9fcd-89556c9690a9/54835b05-573d-4299-97f2-a5366b1fd616"
@@
 		(dnp no)
 		(fields_autoplaced yes)
-		(property "Reference" "#PWR03"
+		(property "Reference" "#PWR?"
 			(at 125.73 128.905 0)
 			(effects
@@
 		)
 		(instances
+			(project "Potencia"
+				(path "/82bf9682-9f8b-46a0-adc6-e19c50674fc0"
+					(reference "#PWR?")
+					(unit 1)
+				)
+			)
 			(project ""
 				(path "/83fe8808-b70b-463e-9fcd-89556c9690a9/54835b05-573d-4299-97f2-a5366b1fd616"
@@
 		)
 	)
+	(sheet_instances
+		(path "/"
+			(page "1")
+		)
+	)
+	(embedded_fonts no)
 )

Commit message: BOMBAS Y FINAL DEL CARRERA
Parts:
- removed K?: EE2-3NKX, Relay_SMD:Relay_DPDT_Kemet_EE2_NUX_NKX, symbol Relay:EE2-3NKX
- added HEATER, R1: R, symbol Device:R
- added K1: DIPxx-1Axx-12xD, Relay_THT:Relay_StandexMeder_DIP_LowProfile, symbol Relay:DIPxx-1Axx-12xD
- added K2: G6K-2, symbol Relay:G6K-2
- added Q1: NPN, symbol Simulation_SPICE:NPN
- added SW1, SW2: SW_SPST, symbol Switch:SW_SPST
- added U1: LM393, symbol Comparator:LM393
Connections:
- net GND: now also HEATER.2, Q1.3 (E)
- net VDD: now also D?.1 (K), K1.13, K1.2, K1.7, K1.8, K2.1, K2.3, K2.6
- net at D?.2 (A), Q?.1 (C): now also K2.8
- net at M?.1 (+): now also K2.7
- net at M?.1 (+): now also K2.4
- new net: Q1.2 (B), R1.2
- new net: HEATER.1, K1.1, K1.14
- new net: K1.6, Q1.1 (C)
- no-connect marks 0 -> 2
Other:
- moved on the sheet: 1k, D?, M?, Q?, U?
