File: KiCad/projecte_neteja_parabrises/Botonera.kicad_sch (KiCad schematic)
At the start: 4 parts, among them SW1 CALEFACTOR, SW2 BOMBAS, SW5 SW_Rotary_1x5_MP

Commit message: SCH ALIMETNACION
Parts:
- removed R3: R, symbol Device:R
Connections:
- net GND: now also SW2.2
Changed lines of the file:
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@@
 	(wire
 		(pts
-			(xy 123.825 85.09) (xy 136.525 85.09)
+			(xy 123.825 85.09) (xy 147.955 85.09)
 		)
 		(stroke
@@
 		(pts
 			(xy 129.54 113.03) (xy 129.54 111.76)
-		)
-		(stroke
-			(width 0)
-			(type default)
-		)
-	)
-	(wire
-		(pts
-			(xy 144.145 85.09) (xy 147.955 85.09)
 		)
 		(stroke
@@
 					(unit 1)
 				)
-			)
-		)
-	)
-	(symbol
-		(lib_id "Device:R")
-		(at 140.335 85.09 90)
-		(unit 1)
-		(exclude_from_sim no)
-		(in_bom yes)
-		(on_board yes)
-		(dnp no)
-		(property "Reference" "R3"
-			(at 140.335 66.04 90)
-			(effects
-				(font
-					(size 1.27 1.27)
-				)
-			)
-		)
-		(property "Value" "R"
-			(at 140.335 68.58 90)
-			(effects
-				(font
-					(size 1.27 1.27)
-				)
-			)
-		)
-		(property "Footprint" ""
-			(at 140.335 86.868 90)
-			(effects
-				(font
-					(size 1.27 1.27)
-				)
-				(hide yes)
-			)
-		)
-		(property "Datasheet" "~"
-			(at 140.335 85.09 0)
-			(effects
-				(font
-					(size 1.27 1.27)
-				)
-				(hide yes)
-			)
-		)
-		(property "Description" "Resistor"
-			(at 140.335 85.09 0)
-			(effects
-				(font
-					(size 1.27 1.27)
-				)
-				(hide yes)
-			)
-		)
-		(pin "2"
-		)
-		(pin "1"
-		)
-		(instances
-			(project ""
-				(path "/83fe8808-b70b-463e-9fcd-89556c9690a9/3042c433-3fca-444b-8551-ace7b9d4faf6"
-					(reference "R3")
-					(unit 1)
-				)

Commit message: ESQUEMATICO V2
Parts:
- removed SW1: CALEFACTOR, Button_Switch_SMD:SW_Push_1P1T_NO_E-Switch_TL3301NxxxxxG, symbol Switch:SW_Push
- removed SW2: BOMBAS, Button_Switch_SMD:SW_Push_1P1T_NO_E-Switch_TL3301NxxxxxG, symbol Switch:SW_Push
- removed SW5: SW_Rotary_1x5_MP, symbol Switch:SW_Rotary_1x5_MP
Connections:
- no-connect marks 1 -> 0

Commit message: alimentacion
Parts:
- added SW1, SW2: SW_Push, Button_Switch_SMD:SW_Push_1P1T_NO_E-Switch_TL3301NxxxxxG, symbol Switch:SW_Push
- added SW3: SW_SP4T_NR01104, Button_Switch_THT:SW_NKK_NR01, symbol Switch:SW_SP4T_NR01104
- added SW4: SW_Rotary_1x4_MP, symbol Switch:SW_Rotary_1x4_MP

Commit message: botonera
Parts:
- removed SW3: SW_SP4T_NR01104, Button_Switch_THT:SW_NKK_NR01, symbol Switch:SW_SP4T_NR01104
- removed SW4: SW_Rotary_1x4_MP, symbol Switch:SW_Rotary_1x4_MP
- added SW5: SW_Rotary_1x5_MP, symbol Switch:SW_Rotary_1x5_MP
Connections:
- new net GND: SW5.1
- no-connect marks 0 -> 1
Changed lines of the file:
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@@
 	(generator_version "9.0")
 	(paper "A4")
-	(symbol
-		(lib_id "Switch:SW_Rotary_1x4_MP")
-		(at 134.62 96.52 0)
-		(unit 1)
-		(exclude_from_sim no)
-		(in_bom yes)
-		(on_board yes)
-		(dnp no)
-		(fields_autoplaced yes)
-		(property "Reference" "SW4"
-			(at 134.62 85.09 0)
-			(effects
-				(font
-					(size 1.27 1.27)
-				)
-			)
-		)
-		(property "Value" "SW_Rotary_1x4_MP"
-			(at 134.62 87.63 0)
-			(effects
-				(font
-					(size 1.27 1.27)
-				)
-			)
-		)
-		(property "Footprint" ""
-			(at 134.62 106.68 0)
-			(effects
-				(font
-					(size 1.27 1.27)
-				)
-				(hide yes)
-			)
-		)
-		(property "Datasheet" "~"
-			(at 134.62 109.22 0)
-			(effects
-				(font
-					(size 1.27 1.27)
-				)
-				(hide yes)
-			)
-		)
-		(property "Description" "Rotary switch 1x4, SP4T with mount point"
-			(at 134.62 96.52 0)
-			(effects
-				(font
-					(size 1.27 1.27)
-				)
-				(hide yes)
-			)
-		)
-		(pin "2"
-		)
-		(pin "4"
-		)
-		(pin "MP"
-		)
-		(pin "1"
-		)
-		(pin "5"
-		)
-		(pin "3"
-		)
-		(instances
-			(project ""
-				(path "/83fe8808-b70b-463e-9fcd-89556c9690a9/3042c433-3fca-444b-8551-ace7b9d4faf6"
-					(reference "SW4")
-					(unit 1)
-				)
-			)
+	(no_connect
+		(at 92.71 100.33)
+	)
+	(wire
+		(pts
+			(xy 107.95 90.17) (xy 109.22 90.17)
+		)
+		(stroke
+			(width 0)
+			(type default)
 		)
 	)
@@
 	)
 	(symbol
+		(lib_id "power:GND")
+		(at 109.22 90.17 90)
+		(unit 1)
+		(exclude_from_sim no)
+		(in_bom yes)
+		(on_board yes)
+		(dnp no)
+		(fields_autoplaced yes)
+		(property "Reference" "#PWR04"
+			(at 115.57 90.17 0)
+			(effects
+				(font
+					(size 1.27 1.27)
+				)
+				(hide yes)
+			)
+		)
+		(property "Value" "GND"
+			(at 113.03 90.1699 90)
+			(effects
+				(font
+					(size 1.27 1.27)
+				)
+				(justify right)
+			)
+		)
+		(property "Footprint" ""
+			(at 109.22 90.17 0)
+			(effects
+				(font
+					(size 1.27 1.27)
+				)
+				(hide yes)
+			)
+		)
+		(property "Datasheet" ""
+			(at 109.22 90.17 0)
+			(effects
+				(font
+					(size 1.27 1.27)
+				)
+				(hide yes)
+			)
+		)
+		(property "Description" "Power symbol creates a global label with name \"GND\" , ground"
+			(at 109.22 90.17 0)
+			(effects
+				(font
+					(size 1.27 1.27)
+				)
+				(hide yes)
+			)
+		)
+		(pin "1"
+		)
+		(instances
+			(project ""
+				(path "/83fe8808-b70b-463e-9fcd-89556c9690a9/3042c433-3fca-444b-8551-ace7b9d4faf6"
+					(reference "#PWR04")
+					(unit 1)
+				)
+			)
+		)
+	)
+	(symbol
 		(lib_id "Switch:SW_Push")
 		(at 118.11 73.66 0)
@@
 	)
 	(symbol
-		(lib_id "Switch:SW_SP4T_NR01104")
-		(at 101.6 93.98 0)
+		(lib_id "Switch:SW_Rotary_1x5_MP")
+		(at 100.33 95.25 0)
 		(unit 1)
 		(exclude_from_sim no)
@@
 		(dnp no)
 		(fields_autoplaced yes)
-		(property "Reference" "SW3"
-			(at 101.6 82.55 0)
-			(effects
-				(font
-					(size 1.27 1.27)
-				)
-			)
-		)
-		(property "Value" "SW_SP4T_NR01104"
-			(at 101.6 85.09 0)
-			(effects
-				(font
-					(size 1.27 1.27)
-				)
-			)
-		)
-		(property "Footprint" "Button_Switch_THT:SW_NKK_NR01"
-			(at 101.6 104.14 0)
-			(effects
-				(font
-					(size 1.27 1.27)
-				)
-				(hide yes)
-			)
-		)
-		(property "Datasheet" "https://www.nkkswitches.com/pdf/NR01%20Rotaries.pdf"
-			(at 101.6 106.68 0)
-			(effects
-				(font
-					(size 1.27 1.27)
-				)
-				(hide yes)
-			)
-		)
-		(property "Description" "NKK Switches NR01 Series rotary SP4T switch"
-			(at 101.6 93.98 0)
-			(effects
-				(font
-					(size 1.27 1.27)
-				)
-				(hide yes)
-			)
+		(property "Reference" "SW5"
+			(at 100.33 83.82 0)
+			(effects
+				(font
+					(size 1.27 1.27)
+				)
+			)
+		)
+		(property "Value" "SW_Rotary_1x5_MP"
+			(at 100.33 86.36 0)
+			(effects
+				(font
+					(size 1.27 1.27)
+				)
+			)
+		)
+		(property "Footprint" ""
+			(at 100.33 105.41 0)
+			(effects
+				(font
+					(size 1.27 1.27)
+				)
+				(hide yes)
+			)
+		)
+		(property "Datasheet" "~"
+			(at 100.33 107.95 0)
+			(effects
+				(font
+					(size 1.27 1.27)
+				)
+				(hide yes)
+			)
+		)
+		(property "Description" "Rotary switch 1x5, SP5T with mount point"
+			(at 100.33 95.25 0)
+			(effects
+				(font
+					(size 1.27 1.27)
+				)
+				(hide yes)
+			)
+		)
+		(pin "1"
+		)
+		(pin "2"
+		)
+		(pin "MP"
+		)
+		(pin "3"
+		)
+		(pin "4"
+		)
+		(pin "6"
 		)
 		(pin "5"
 		)
-		(pin "3"
-		)
-		(pin "MP"
-		)
-		(pin "1"
-		)
-		(pin "C"
-		)
-		(pin "2"
-		)
-		(pin "4"
-		)
 		(instances
 			(project ""
 				(path "/83fe8808-b70b-463e-9fcd-89556c9690a9/3042c433-3fca-444b-8551-ace7b9d4faf6"
-					(reference "SW3")
-					(unit 1)
-				)
+					(reference "SW5")
+					(unit 1)
+				)

Commit message: botonera
Parts:
- added R2, R3: R, symbol Device:R
Connections:
- net GND: now also R2.2, R3.2
- net 5V: now reaches SW2.1
- net 5V: now also SW1.1, SW5.6
- net at SW2.2: now also R2.1
- net at SW1.2: now also R3.1
Other:
- moved on the sheet: SW5

Commit message: SCH V1
Parts:
- removed R2: R, symbol Device:R
- SW1: renamed from SW2; value SW_Push -> CALEFACTOR
- SW2: renamed from SW1; value SW_Push -> BOMBAS
Connections:
- net GND: now also SW1.2, SW5.6; no longer SW5.1
- net SW2: now reaches SW5.2
- net SW2: now also SW2.1
- net SW3: now reaches SW5.3
- net SW4: now reaches SW5.4
- net SW5: now reaches SW5.5
- removed net 5V: SW1.1, SW2.1, SW5.6
- new net SW1: SW1.1, SW5.1
Other:
- moved on the sheet: R3, SW1, SW2, SW5
