File: KiCad/projecte_neteja_parabrises/untitled.kicad_sch (KiCad schematic)
At the start: 14 parts, among them J2 DE9_Pins, J3 DE9_Pins, SW1 CALEFACTOR, SW2 BOMBAS, SW3 SW_SP5T_NR01105, U8 TJA1049TK-3, U9 MAX232

Commit message: Actualizacion errores
Changed lines of the file:
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@@
 	)
 	(global_label "CANRX"
-		(shape input)
+		(shape output)
 		(at 193.04 65.405 180)
 		(fields_autoplaced yes)
@@
 	)
 	(global_label "RX"
-		(shape input)
+		(shape output)
 		(at 34.29 74.93 180)
 		(fields_autoplaced yes)
