File: KiCad/projecte_neteja_parabrises/Microcontrolador.kicad_sch (KiCad schematic)
At the start: 16 parts, among them U5 PIC24HJ32GP502, U6 HDC2080, U7 SN74LVC2T45DCUR, Y1 Crystal

Commit message: MCLR
Parts:
- removed C16: 100n, Capacitor_SMD:C_0805_2012Metric, symbol Device:C
- added D2: LED, symbol Device:LED
- added J1: Conn_01x05_Pin, symbol Connector:Conn_01x05_Pin
- added JP1: Jumper_3_Bridged12, symbol Jumper:Jumper_3_Bridged12
- added R13, R14: 470, symbol Device:R
- added SW4: SW_Omron_B3FS, symbol Switch:SW_Omron_B3FS
- R10, R11, R12: value R -> 4,7k
- R7: value 470 -> R; footprint Resistor_SMD:R_0603_1608Metric_Pad0.98x0.95mm_HandSolder -> (none)
- R8: value 10K -> R; footprint Resistor_SMD:R_0603_1608Metric_Pad0.98x0.95mm_HandSolder -> (none)
- R9: value R -> 10k
Connections:
- net GND: now also R8.1, J1.3 (Pin_3), SW4.2
- net MCLR: now also JP1.2 (C); no longer R7.2
- net VDD: no longer R8.2
- net at R7.1: now also JP1.3 (B); no longer R8.1
- net PWM: no longer names the net of U5.16 (RB7)
- net PWM: now also R13.1
- net SW5: no longer names the net of U5.15 (RB6)
- net SW5: now also R14.1
- new net: R7.2, SW4.1
- new net: J1.1 (Pin_1), JP1.1 (A)
- new net: D2.1 (K), R8.2
- new net PGC: J1.5 (Pin_5), R14.2
- new net PGD: J1.4 (Pin_4), R13.2
- new net VCC: D2.2 (A), J1.2 (Pin_2)

Commit message: arreglos
Parts:
- JP1: footprint (none) -> Connector_PinHeader_2.54mm:PinHeader_1x03_P2.54mm_Vertical
- R7, R8: footprint (none) -> Resistor_SMD:R_0603_1608Metric_Pad0.98x0.95mm_HandSolder
- SW4: footprint (none) -> Button_Switch_SMD:SW_SPST_Omron_B3FS-100xP
Changed lines of the file:
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@@
 			)
 		)
-		(property "Footprint" ""
+		(property "Footprint" "Button_Switch_SMD:SW_SPST_Omron_B3FS-100xP"
 			(at 80.645 19.05 0)
 			(effects
@@
 			)
 		)
-		(property "Footprint" ""
+		(property "Footprint" "Connector_PinHeader_2.54mm:PinHeader_1x03_P2.54mm_Vertical"
 			(at 53.34 24.13 0)
 			(effects
@@
 			)
 		)
-		(property "Footprint" ""
+		(property "Footprint" "Resistor_SMD:R_0603_1608Metric_Pad0.98x0.95mm_HandSolder"
 			(at 26.035 116.713 90)
 			(effects
@@
 			)
 		)
-		(property "Footprint" ""
+		(property "Footprint" "Resistor_SMD:R_0603_1608Metric_Pad0.98x0.95mm_HandSolder"
 			(at 71.755 25.908 90)
 			(effects

Commit message: Placa definitiva
Parts:
- D2: footprint (none) -> LED_SMD:LED_0805_2012Metric_Pad1.15x1.40mm_HandSolder
- J1: footprint (none) -> Connector_PinHeader_2.54mm:PinHeader_1x05_P2.54mm_Vertical
- R13, R14: footprint (none) -> Resistor_SMD:R_0603_1608Metric_Pad0.98x0.95mm_HandSolder
Connections:
- net PWM2 is gone; now on net FC1: U5.21 (RB10)
- net FC1: no longer U5.12 (RA4)
- net SW4: now also U5.12 (RA4); no longer U5.14 (RB5)
- new net SW5: U5.14 (RB5)
Other:
- moved on the sheet: C2
Changed lines of the file:
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@@
 	(wire
 		(pts
-			(xy 20.32 80.645) (xy 29.21 80.645)
+			(xy 20.32 80.01) (xy 27.94 80.01)
 		)
 		(stroke
@@
 	(wire
 		(pts
-			(xy 36.83 80.645) (xy 45.085 80.645)
-		)
-		(stroke
-			(width 0)
-			(type default)
-		)
-	)
-	(wire
-		(pts
 			(xy 84.455 85.09) (xy 85.725 85.09)
 		)
@@
 	(wire
 		(pts
-			(xy 45.085 80.01) (xy 47.625 80.01)
-		)
-		(stroke
-			(width 0)
-			(type default)
-		)
-	)
-	(wire
-		(pts
 			(xy 97.155 110.49) (xy 101.6 110.49)
 		)
@@
 	(wire
 		(pts
-			(xy 20.32 82.55) (xy 20.32 80.645)
+			(xy 20.32 82.55) (xy 20.32 80.01)
 		)
 		(stroke
@@
 	(wire
 		(pts
+			(xy 35.56 80.01) (xy 47.625 80.01)
+		)
+		(stroke
+			(width 0)
+			(type default)
+		)
+	)
+	(wire
+		(pts
 			(xy 85.09 110.49) (xy 89.535 110.49)
 		)
@@
 	(wire
 		(pts
-			(xy 45.085 80.645) (xy 45.085 80.01)
-		)
-		(stroke
-			(width 0)
-			(type default)
-		)
-	)
-	(wire
-		(pts
 			(xy 153.035 39.37) (xy 153.035 41.91)
 		)
@@
 	(global_label "FC1"
 		(shape input)
-		(at 40.64 93.98 180)
+		(at 94.615 80.01 0)
 		(fields_autoplaced yes)
 		(effects
@@
 				(size 1.27 1.27)
 			)
-			(justify right)
+			(justify left)
 		)
 		(property "Intersheetrefs" "${INTERSHEET_REFS}"
-			(at 34.0867 93.98 0)
+			(at 101.1683 80.01 0)
 			(effects
 				(font
 					(size 1.27 1.27)
 				)
-				(justify right)
+				(justify left)
 				(hide yes)
 			)
@@
 	(global_label "PWM2"
 		(shape input)
-		(at 94.615 80.01 0)
+		(at 97.79 110.49 270)
 		(fields_autoplaced yes)
 		(effects
@@
 				(size 1.27 1.27)
 			)
-			(justify left)
+			(justify right)
 		)
 		(property "Intersheetrefs" "${INTERSHEET_REFS}"
-			(at 102.9825 80.01 0)
+			(at 97.79 118.8575 90)
 			(effects
 				(font
 					(size 1.27 1.27)
 				)
-				(justify left)
+				(justify right)
 				(hide yes)
 			)
@@
 	(global_label "SW4"
 		(shape input)
-		(at 41.91 102.235 180)
+		(at 40.64 93.98 180)
 		(fields_autoplaced yes)
 		(effects
@@
 		)
 		(property "Intersheetrefs" "${INTERSHEET_REFS}"
-			(at 35.0544 102.235 0)
+			(at 33.7844 93.98 0)
 			(effects
 				(font
@@
 	(global_label "SW5"
 		(shape input)
-		(at 99.06 110.49 270)
+		(at 41.91 102.235 180)
 		(fields_autoplaced yes)
 		(effects
@@
 		)
 		(property "Intersheetrefs" "${INTERSHEET_REFS}"
-			(at 99.06 117.3456 90)
+			(at 35.0544 102.235 0)
 			(effects
 				(font
@@
 			)
 		)
-		(property "Footprint" ""
+		(property "Footprint" "Resistor_SMD:R_0603_1608Metric_Pad0.98x0.95mm_HandSolder"
 			(at 93.345 112.268 90)
 			(effects
@@
 			)
 		)
-		(property "Footprint" ""
+		(property "Footprint" "Resistor_SMD:R_0603_1608Metric_Pad0.98x0.95mm_HandSolder"
 			(at 94.615 95.123 90)
 			(effects
@@
 			)
 		)
-		(property "Footprint" ""
+		(property "Footprint" "LED_SMD:LED_0805_2012Metric_Pad1.15x1.40mm_HandSolder"
 			(at 33.655 114.935 0)
 			(effects
@@
 			)
 		)
-		(property "Footprint" ""
+		(property "Footprint" "Connector_PinHeader_2.54mm:PinHeader_1x05_P2.54mm_Vertical"
 			(at 24.13 33.655 0)
 			(effects
@@
 	(symbol
 		(lib_id "Device:C")
-		(at 33.02 80.645 90)
+		(at 31.75 80.01 90)
 		(unit 1)
 		(exclude_from_sim no)
@@
 		(dnp no)
 		(property "Reference" "C2"
-			(at 36.195 79.375 90)
+			(at 34.925 78.74 90)
 			(effects
 				(font
@@
 		)
 		(property "Value" "100n"
-			(at 33.02 83.82 90)
+			(at 31.75 83.185 90)
 			(effects
 				(font
@@
 		)
 		(property "Footprint" "Capacitor_SMD:C_0805_2012Metric"
-			(at 36.83 79.6798 0)
+			(at 35.56 79.0448 0)
 			(effects
 				(font
@@
 		)
 		(property "Datasheet" "~"
-			(at 33.02 80.645 0)
+			(at 31.75 80.01 0)
 			(effects
 				(font
@@
 		)
 		(property "Description" "Unpolarized capacitor"
-			(at 33.02 80.645 0)
+			(at 31.75 80.01 0)
 			(effects
 				(font

Commit message: Actualizacion errores
Parts:
- removed R11, R12: 4,7k, Resistor_SMD:R_0603_1608Metric_Pad0.98x0.95mm_HandSolder, symbol Device:R
- removed U7: SN74LVC2T45DCUR, Package_SO:VSSOP-8_2.3x2mm_P0.5mm, symbol Logic_LevelTranslator:SN74LVC2T45DCUR
- R7, R8: value R -> 1k
Connections:
- net GND: no longer R10.1, R9.2
- net SCL: now also R9.2, U6.6 (SCL)
- net SDA: now also U6.1 (SDA)
- net VDD: now also R10.2, R9.1, U6.5 (VDD)
Other:
- moved on the sheet: R10, R9, U6

Commit message: Led
Parts:
- removed D2: LED, LED_SMD:LED_0805_2012Metric_Pad1.15x1.40mm_HandSolder, symbol Device:LED
- removed R8: 1k, Resistor_SMD:R_0603_1608Metric_Pad0.98x0.95mm_HandSolder, symbol Device:R
Connections:
- net VCC is gone; now on net VDD: J1.2 (Pin_2)

Commit message: Botonera
Changed lines of the file:
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@@
-	(wire
-		(pts
-			(xy 22.86 77.47) (xy 47.625 77.47)
-		)
-		(stroke
-			(width 0)
-			(type default)
-		)
-	)
 	(wire
 		(pts
@@
 				)
 				(justify left)
+				(hide yes)
+			)
+		)
+	)
+	(global_label "SW5"
+		(shape input)
+		(at 41.91 102.235 180)
+		(fields_autoplaced yes)
+		(effects
+			(font
+				(size 1.27 1.27)
+			)
+			(justify right)
+		)
+		(property "Intersheetrefs" "${INTERSHEET_REFS}"
+			(at 35.0544 102.235 0)
+			(effects
+				(font
+					(size 1.27 1.27)
+				)
+				(justify right)
 				(hide yes)
 			)
@@
 		)
 	)
+	(global_label "SW3"
+		(shape input)
+		(at 36.195 91.44 180)
+		(fields_autoplaced yes)
+		(effects
+			(font
+				(size 1.27 1.27)
+			)
+			(justify right)
+		)
+		(property "Intersheetrefs" "${INTERSHEET_REFS}"
+			(at 29.3394 91.44 0)
+			(effects
+				(font
+					(size 1.27 1.27)
+				)
+				(justify right)
+				(hide yes)
+			)
+		)
+	)
 	(global_label "FC1"
 		(shape input)
@@
 				)
 				(justify left)
+				(hide yes)
+			)
+		)
+	)
+	(global_label "SW1"
+		(shape input)
+		(at 30.48 74.93 180)
+		(fields_autoplaced yes)
+		(effects
+			(font
+				(size 1.27 1.27)
+			)
+			(justify right)
+		)
+		(property "Intersheetrefs" "${INTERSHEET_REFS}"
+			(at 23.6244 74.93 0)
+			(effects
+				(font
+					(size 1.27 1.27)
+				)
+				(justify right)
 				(hide yes)
 			)
@@
 		)
 	)
+	(global_label "GATE B"
+		(shape input)
+		(at 42.545 58.42 180)
+		(fields_autoplaced yes)
+		(effects
+			(font
+				(size 1.27 1.27)
+			)
+			(justify right)
+		)
+		(property "Intersheetrefs" "${INTERSHEET_REFS}"
+			(at 32.847 58.42 0)
+			(effects
+				(font
+					(size 1.27 1.27)
+				)
+				(justify right)
+				(hide yes)
+			)
+		)
+	)
+	(global_label "CANRX"
+		(shape input)
+		(at 94.615 74.93 0)
+		(fields_autoplaced yes)
+		(effects
+			(font
+				(size 1.27 1.27)
+			)
+			(justify left)
+		)
+		(property "Intersheetrefs" "${INTERSHEET_REFS}"
+			(at 103.7688 74.93 0)
+			(effects
+				(font
+					(size 1.27 1.27)
+				)
+				(justify left)
+				(hide yes)
+			)
+		)
+	)
 	(global_label "SW4"
 		(shape input)
@@
 				)
 				(justify right)
-				(hide yes)
-			)
-		)
-	)
-	(global_label "SW5"
-		(shape input)
-		(at 41.91 102.235 180)
-		(fields_autoplaced yes)
-		(effects
-			(font
-				(size 1.27 1.27)
-			)
-			(justify right)
-		)
-		(property "Intersheetrefs" "${INTERSHEET_REFS}"
-			(at 35.0544 102.235 0)
-			(effects
-				(font
-					(size 1.27 1.27)
-				)
-				(justify right)
-				(hide yes)
-			)
-		)
-	)
-	(global_label "SW2"
-		(shape input)
-		(at 22.86 77.47 180)
-		(fields_autoplaced yes)
-		(effects
-			(font
-				(size 1.27 1.27)
-			)
-			(justify right)
-		)
-		(property "Intersheetrefs" "${INTERSHEET_REFS}"
-			(at 16.0044 77.47 0)
-			(effects
-				(font
-					(size 1.27 1.27)
-				)
-				(justify right)
-				(hide yes)
-			)
-		)
-	)
-	(global_label "GATE B"
-		(shape input)
-		(at 42.545 58.42 180)
-		(fields_autoplaced yes)
-		(effects
-			(font
-				(size 1.27 1.27)
-			)
-			(justify right)
-		)
-		(property "Intersheetrefs" "${INTERSHEET_REFS}"
-			(at 32.847 58.42 0)
-			(effects
-				(font
-					(size 1.27 1.27)
-				)
-				(justify right)
-				(hide yes)
-			)
-		)
-	)
-	(global_label "CANRX"
-		(shape input)
-		(at 94.615 74.93 0)
-		(fields_autoplaced yes)
-		(effects
-			(font
-				(size 1.27 1.27)
-			)
-			(justify left)
-		)
-		(property "Intersheetrefs" "${INTERSHEET_REFS}"
-			(at 103.7688 74.93 0)
-			(effects
-				(font
-					(size 1.27 1.27)
-				)
-				(justify left)
 				(hide yes)
 			)
@@
 		)
 	)
-	(global_label "SW1"
-		(shape input)
-		(at 30.48 74.93 180)
+	(global_label "MCLR"
+		(shape input)
+		(at 53.34 27.94 270)
 		(fields_autoplaced yes)
 		(effects
@@
 		)
 		(property "Intersheetrefs" "${INTERSHEET_REFS}"
-			(at 23.6244 74.93 0)
+			(at 53.34 35.9447 90)
 			(effects
 				(font
@@
 		)
 	)
-	(global_label "MCLR"
-		(shape input)
-		(at 53.34 27.94 270)
+	(global_label "RX"
+		(shape input)
+		(at 94.615 66.04 0)
+		(fields_autoplaced yes)
+		(effects
+			(font
+				(size 1.27 1.27)
+			)
+			(justify left)
+		)
+		(property "Intersheetrefs" "${INTERSHEET_REFS}"
+			(at 100.0797 66.04 0)
+			(effects
+				(font
+					(size 1.27 1.27)
+				)
+				(justify left)
+				(hide yes)
+			)
+		)
+	)
+	(global_label "SW2"
+		(shape input)
+		(at 47.625 77.47 180)
 		(fields_autoplaced yes)
 		(effects
@@
 		)
 		(property "Intersheetrefs" "${INTERSHEET_REFS}"
-			(at 53.34 35.9447 90)
+			(at 40.7694 77.47 0)
 			(effects
 				(font
@@
 				)
 				(justify right)
-				(hide yes)
-			)
-		)
-	)
-	(global_label "SW3"
-		(shape input)
-		(at 36.195 91.44 180)
-		(fields_autoplaced yes)
-		(effects
-			(font
-				(size 1.27 1.27)
-			)
-			(justify right)
-		)
-		(property "Intersheetrefs" "${INTERSHEET_REFS}"
-			(at 29.3394 91.44 0)
-			(effects
-				(font
-					(size 1.27 1.27)
-				)
-				(justify right)
-				(hide yes)
-			)
-		)
-	)
-	(global_label "RX"
-		(shape input)
-		(at 94.615 66.04 0)
-		(fields_autoplaced yes)
-		(effects
-			(font
-				(size 1.27 1.27)
-			)
-			(justify left)
-		)
-		(property "Intersheetrefs" "${INTERSHEET_REFS}"
-			(at 100.0797 66.04 0)
-			(effects
-				(font
-					(size 1.27 1.27)
-				)
-				(justify left)
 				(hide yes)
 			)
@@
 		(on_board yes)
 		(dnp no)
-		(fields_autoplaced yes)
 		(property "Reference" "#PWR010"
 			(at 20.32 88.9 0)

Commit message: POTENCIA GND
Parts:
- removed R13, R14: 470, Resistor_SMD:R_0603_1608Metric_Pad0.98x0.95mm_HandSolder, symbol Device:R
Connections:
- net SW4 is gone; now on net FC1: U5.12 (RA4)
- net SW5 is gone; now on net FC2: U5.14 (RB5)
- net FC1: no longer U5.21 (RB10)
- net FC2: no longer U5.24 (RP13)
- net PGC: now also U5.15 (RB6)
- net PGD: now also U5.16 (RB7)
- net SDA: now also R10.1
- new net PWM: U5.21 (RB10)
- new net PWM2: U5.24 (RP13)
Other:
- moved on the sheet: R10

Commit message: micro
Parts:
- removed U5: PIC24HJ32GP502, Package_SO:SOIC-28W_7.5x17.9mm_P1.27mm, symbol New_Library_0:PIC24HJ32GP302/304
- added 11: PIC24HJ64GP504, symbol New_Library_0:PIC24HJ64GP504
- renumbered C17 to C4, C3 to C5, C4 to C6, R10 to R1, R9 to R2, R7 to R3, SW4 to SW1, U6 to U3
Connections:
- net CANRX: now also 11.36 (RP19)
- net CANTX: now also 11.37 (RP20)
- net FC1: now also 11.32 (RA8)
- net FC2: now also 11.33 (RB4)
- net GATE B: now also 11.25 (RC0)
- net GATE C: now also 11.27 (RC2)
- net GND: now also 11.16 (AVss), 11.6 (VSS)
- net MCLR: now also 11.18 (~{MCLR})
- net OSC1: now also 11.30 (OSCI)
- net OSC2: now also 11.31 (OSC2)
- net PGC: now also 11.9 (PGEC2)
- net PGD: now also 11.8 (PGED2)
- net PWM: now also 11.21 (RP0)
- net PWM2: now also 11.22 (RP1)
- net RX: now also 11.23 (RP2)
- net SCL: now also 11.44 (SCL1)
- net SDA: now also 11.1 (SDA1)
- net SW1: now also 11.2 (RC6)
- net SW2: now also 11.3 (RC7)
- net SW3: now also 11.4 (RC8)
- net SWB: now also 11.20 (RA1)
- net SWC: now also 11.19 (RA0)
- net TX: now also 11.24 (RP3)
- net VDD: now also 11.28 (Vdd), 11.40 (Vdd)
- net at C4.1: now also 11.7 (VCAP)
- net at C1.1: now also 11.17 (AVdd)
- net at C2.2: now also 11.29 (Vss)
- no-connect marks 1 -> 16
Other:
- moved on the sheet: C1, C2, C4, J1, JP1, R3, SW1
