File: KiCad/projecte_neteja_parabrises/Alimentación.kicad_sch (KiCad schematic)
At the start: 14 parts, among them J4 Conn_01x02_Pin, U1 LM1117DT-3.3, U2 LM2596S-5

Commit message: pcb
Parts:
- added TP1, TP2, TP3: TestPoint, TestPoint:TestPoint_Keystone_5015_Micro_Mini, symbol Connector:TestPoint
Connections:
- net 5V: now also TP2.1
- net VDD: now also TP3.1
- net Vbat: now also TP1.1

Commit message: pcb
Connections:
- net Vbat renamed 12V
Changed lines of the file:
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@@
 		)
 	)
-	(global_label "Vbat"
+	(global_label "12V"
 		(shape input)
 		(at 32.766 79.502 0)
@@
 		)
 		(property "Intersheetrefs" "${INTERSHEET_REFS}"
-			(at 39.8635 79.502 0)
+			(at 39.2588 79.502 0)
 			(effects
 				(font
@@
 		)
 	)
-	(global_label "Vbat"
+	(global_label "12V"
 		(shape input)
 		(at 59.69 80.01 180)
@@
 		)
 		(property "Intersheetrefs" "${INTERSHEET_REFS}"
-			(at 52.5925 80.01 0)
+			(at 53.1972 80.01 0)
 			(effects
 				(font
@@
 		)
 		(instances
+			(project "Alimentación"
+				(path "/2ad4f79a-6f2e-459e-be48-40e5d52d2cdd"
+					(reference "TP?")
+					(unit 1)
+				)
+			)
 			(project ""
 				(path "/83fe8808-b70b-463e-9fcd-89556c9690a9/a8962c48-b3a9-4541-b459-e1566624b900"
@@
 		)
 		(instances
+			(project "Alimentación"
+				(path "/2ad4f79a-6f2e-459e-be48-40e5d52d2cdd"
+					(reference "TP?")
+					(unit 1)
+				)
+			)
 			(project ""
 				(path "/83fe8808-b70b-463e-9fcd-89556c9690a9/a8962c48-b3a9-4541-b459-e1566624b900"
@@
 		)
 		(instances
-			(project ""
-				(path "/83fe8808-b70b-463e-9fcd-89556c9690a9/a8962c48-b3a9-4541-b459-e1566624b900"
+			(project "Alimentación"
+				(path "/2ad4f79a-6f2e-459e-be48-40e5d52d2cdd"
+					(reference "TP?")
+					(unit 1)
+				)
+			)
+			(project ""
+				(path "/83fe8808-b70b-463e-9fcd-89556c9690a9/a8962c48-b3a9-4541-b459-e1566624b900"
