File: KiCad/projecte_neteja_parabrises/projecte_neteja_parabrises.kicad_pcb (KiCad board)
At the start: 2 copper layers, 117.2 x 96.5 mm, 84 parts, among them J1 Conn_01x05_Pin, J2 DE9_Pins, J3 DE9_Pins, J4 Conn_01x02_Pin, K2 Fujitsu_FTR-LYAA005x, K3 Fujitsu_FTR-LYAA005x, K4 Fujitsu_FTR-LYAA005x, M1 Motor_DC, M2 Motor_DC, M3 Motor_DC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

Commit message: pcb
Parts:
- moved C15 58.3 mm to (90.4, 81.2)
- moved C2 23.7 mm to (120.7, 113.7)
- moved D2 17.7 mm to (126.1, 114.6)
- moved R8 17.7 mm to (126.1, 111.8)
- moved R4 2.79 mm to (96.0, 112.9)
- moved R20 2.08 mm to (115.2, 96.1)
- moved R10 1.95 mm to (115.8, 79.2)
- moved C8 1.78 mm to (160.2, 103.8)
- moved C5 1.78 mm to (155.5, 103.8)
- moved C6 1.78 mm to (159.5, 106.8)
- moved C7 1.78 mm to (159.3, 109.5)
- moved U9 1.78 mm to (166.5, 107.0)
- moved C9 1.65 mm to (176.1, 103.4)
Routing:
- net VDD: track 21.3 -> 39.3 mm, vias 1 -> 4
- net Net-(Q3-B): track 7.93 -> 5.03 mm
- net SW3: track 34.5 -> 36.6 mm
- net Net-(U9-T1OUT): track 21.1 -> 23.0 mm
- net GATE C: track 38.5 -> 40.2 mm, vias 0 -> 2
- net Net-(U9-R1IN): track 16.4 -> 17.7 mm
- net CANTX: track 34.5 -> 33.3 mm, vias 0 -> 2
- net SW1: track 32.0 -> 33.0 mm, vias 0 -> 1
- net TX: track 46.4 -> 45.4 mm
- net 5V: track 8.58 -> 9.52 mm
- net RX: track 46.0 -> 45.2 mm
- net GND: track 89.0 -> 89.7 mm
- net CANRX: track 33.1 -> 32.7 mm, vias 0 -> 2
- net FC2: track 54.1 -> 54.3 mm, vias 0 -> 1
- net GATE B2: vias 0 -> 2
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